Commit message: slam-working

File: description/lidar.xacro (robot description, xacro)
@@ -1,8 +1,8 @@
 <?xml version="1.0"?>
-<robot xmlns:xacro="http://www.ros.org/wiki/xacro"  >
+<robot xmlns:xacro="http://www.ros.org/wiki/xacro">
     <joint name="laser_joint" type="fixed">
         <parent link="chassis"/>
         <child link="laser_frame"/>
-        <origin xyz="0.1 0.0 0.15" rpy="0.0 0.0 0.0"/>
+        <origin xyz="0.1 0 0.15" rpy="0 0 0"/>
     </joint>
     <link name="laser_frame">
@@ -10,4 +10,11 @@
             <geometry>
                 <cylinder radius="0.05" length="0.04"/>
+            </geometry>
+            <material name="red"/>
+        </visual>
+        <visual>
+            <origin xyz="0 0 -0.05"/>
+            <geometry>
+                <cylinder radius="0.01" length="0.1"/>
             </geometry>
             <material name="red"/>
@@ -19,5 +26,5 @@
         </collision>
         <xacro:inertial_cylinder mass="0.1" length="0.04" radius="0.125">
-            <origin xyz="0.0 0.0 0.0" rpy="0.0 0.0 0.0"/>
+            <origin xyz="0 0 0" rpy="0 0 0"/>
         </xacro:inertial_cylinder>
     </link>

File: description/robot.urdf.xacro (robot description, xacro)
@@ -2,4 +2,5 @@
 <robot xmlns:xacro="http://www.ros.org/wiki/xacro"  name="robot">
     <xacro:arg name="use_ros2_control" default="true"/>
+    <xacro:arg name="sim_mode" default="false"/>
     <xacro:include filename="robot_core.xacro" />
     <xacro:if value="$(arg use_ros2_control)">

File: description/robot_core.xacro (robot description, xacro)
@@ -75,5 +75,5 @@
         </collision>
         <xacro:inertial_cylinder mass="0.1" length="0.06" radius="0.125">
-            <origin xyz="0.0 0.0 0.0" rpy="0.0 0.0 0.0"/>
+            <origin xyz="0 0 0" rpy="0 0 0"/>
         </xacro:inertial_cylinder>
     </link>
@@ -85,5 +85,5 @@
         <parent link="base_link"/>
         <child link="right_wheel"/>
-        <origin xyz="0 -0.2025 0" rpy="${pi/2} 0.0 0.0"/>
+        <origin xyz="0 -0.2025 0" rpy="${pi/2} 0 0"/>
         <axis xyz="0 0 -1"/>
     </joint>
@@ -101,5 +101,5 @@
         </collision>
         <xacro:inertial_cylinder mass="0.1" length="0.06" radius="0.125">
-            <origin xyz="0.0 0.0 0.0" rpy="0.0 0.0 0.0"/>
+            <origin xyz="0 0 0" rpy="0 0 0"/>
         </xacro:inertial_cylinder>
     </link>
@@ -108,8 +108,8 @@
     </gazebo>
     <!-- CASTER WHEEL LINK -->
-    <joint name="caster_wheel_likn" type="fixed">
+    <joint name="caster_wheel_joint" type="fixed">
         <parent link="chassis"/>
         <child link="caster_wheel"/>
-        <origin xyz="0.10 0.0 0.0" rpy="0.0 0.0 0.0"/>
+        <origin xyz="0.10 0 0" rpy="0 0 0"/>
     </joint>
     <link name="caster_wheel">
@@ -126,5 +126,5 @@
         </collision>
         <xacro:inertial_sphere mass="1" radius="0.125">
-            <origin xyz="0.0 0.0 0.0" rpy="0.0 0.0 0.0"/>
+            <origin xyz="0 0 0" rpy="0 0 0"/>
         </xacro:inertial_sphere>
     </link>

File: description/ros2_control.xacro (robot description, xacro)
@@ -11,5 +11,5 @@
                 <param name="baud_rate">57600</param>
                 <param name="timeout">1000</param>
-                <param name="enc_counts_per_rev">96</param>
+                <param name="enc_counts_per_rev">100</param>
             </hardware>
             <!-- Note everything below here is the same as the Gazebo one -->
